File: prj-kicad/pmod-trh.kicad_pcb (KiCad board)
At the start: 2 copper layers, 38.1 x 20.3 mm, 16 parts, among them P1 PMOD, U1 ATSAMD09C13A, U2 SI7021

Commit message: Hardware: Create rev2, fix known problems of rev1 (UART, reset) and add power control
Parts:
- added C4: 1uF, pmod-trh:SMD0603, F.Cu at (149.0, 111.0)
- added D1: LED, pmod-trh:SMD0805, F.Cu at (144.0, 111.2)
- added Q1: Si2319, pmod-trh:SOT23-3, F.Cu at (156.5, 98.0)
- added R5: 10k, pmod-trh:SMD0603, F.Cu at (149.8, 108.8)
- added R6: 0, pmod-trh:SMD0603, F.Cu at (156.5, 100.5)
- added R7: 10k, pmod-trh:SMD0603, F.Cu at (153.5, 100.5)
- added R8: 330, pmod-trh:SMD0603, F.Cu at (146.5, 112.0)
- moved agilack-11.5 2.50 mm to (146.0, 98.0)
Connections:
- L2 pad 1: +3.3V -> Net-(L2-Pad1)
- P1 pad 1: PMOD_CTS -> unconnected-(P1-Pad1)
- P1 pad 4: PMOD_RTS -> unconnected-(P1-Pad4)
- U1 pad 1: PMOD_TXD -> PWR_SENSOR
- U1 pad 10: PMOD_RTS -> PMOD_TXD
- U1 pad 14: PMOD_RXD -> LED
- U1 pad 9: PMOD_CTS -> PMOD_RXD
Routing:
- net PWR_SENSOR: track 0.00 -> 19.9 mm
- net RST: track 15.4 -> 28.3 mm
- net PMOD_RTS: track 10.7 -> 0.00 mm
- net PMOD_CTS: track 6.53 -> 0.00 mm, vias 1 -> 0
- net PMOD_RXD: track 11.9 -> 5.44 mm
- net PMOD_TXD: track 15.9 -> 10.7 mm
- net Net-(L2-Pad1): track 0.00 -> 4.48 mm
- net +3.3V: track 43.1 -> 47.0 mm
- net LED: track 0.00 -> 3.97 mm
- net Net-(R8-Pad1): track 0.00 -> 1.55 mm
- net GND: track 141.1 -> 142.3 mm, vias 25 -> 26
Other:
- board text added: "rev2"
- board text removed: "rev1"
